Commit message: feat: Add 'anchor module' to arm

File: tutorials/simenv/start_env/robot.urdf (robot description, URDF)
Before this commit: robot robot, 4 links, 3 joints
Links:
- link MODULE_1: geometry visual base_module length=2.0
- link MODULE_2: geometry visual base_module length=1.5
- link MODULE_3: geometry visual base_module length=1.0
- link anchor: geometry visual anchor_module length=0.5
