Commit message: fix: some extra robot urdf's, trained network, speed up when visuals on

File: src/environment/robot1.urdf (robot description, URDF)
Before this commit: robot robot, 5 links, 3 joints
Links:
- removed link MODULE_0
- removed link MODULE_1
- removed link MODULE_2
- removed link MODULE_3
- added link MODULE_1_TILT; visual tilting_module length=2.5
- added link MODULE_2_TILT_ROTATE; visual complex_module length=2.5
- added link MODULE_3_TILT; visual tilting_module length=1.5
Joints:
- joint MODULE_1_JOINT: child MODULE_1 -> MODULE_1_TILT
- joint MODULE_2_JOINT: child MODULE_2 -> MODULE_2_TILT_ROTATE; parent MODULE_1 -> MODULE_1_TILT
- joint MODULE_3_JOINT: child MODULE_3 -> MODULE_3_TILT; parent MODULE_2 -> MODULE_2_TILT_ROTATE

File: src/environment/robot2.urdf (robot description, URDF)
Before this commit: robot robot, 5 links, 3 joints
Links:
- removed link MODULE_0
- removed link MODULE_1
- removed link MODULE_2
- removed link MODULE_3
- added link MODULE_1_TILT; visual tilting_module length=2
- added link MODULE_2_TILT; visual tilting_module length=2
- added link MODULE_3_TILT; visual tilting_module length=1.5
Joints:
- joint MODULE_1_JOINT: child MODULE_1 -> MODULE_1_TILT
- joint MODULE_2_JOINT: child MODULE_2 -> MODULE_2_TILT; parent MODULE_1 -> MODULE_1_TILT
- joint MODULE_3_JOINT: child MODULE_3 -> MODULE_3_TILT; parent MODULE_2 -> MODULE_2_TILT
