Commit message: reset robot

File: src/environment/robot4.urdf (robot description, URDF)
Before this commit: robot robot, 4 links, 3 joints
Links:
- added link MODULE_0; visual tilting_module length=1.5
- link MODULE_1: geometry visual tilting_module length=2.5
- link MODULE_2: geometry visual tilting_module length=2.5
- link MODULE_3: geometry visual complex_module length=2.5
- link anchor: geometry visual anchor_module length=1
