Commit message: Different modules. Builder and Assets complete

File: src/environment/robot.urdf (robot description, URDF)
Before this commit: robot robot, 4 links, 3 joints
Links:
- link MODULE_1: geometry visual tilting_module length=1.5
- link MODULE_2: geometry visual tilting_module length=1.5
- link MODULE_3: geometry visual tilting_module length=1.5

Commit message: Camera on other side, fix anchor_module height

File: src/environment/robot.urdf (robot description, URDF)
Before this commit: robot robot, 4 links, 3 joints
Links:
- link MODULE_1: geometry visual tilting_module length=1

Commit message: Deep-Q learning neural network (#32)
* feat: add pytorch example code

* feat: implement rought dqn code

* feat: implement rought dqn code

* feat: seperate dqn and dqn-learner code

* fix paths

* add different actions

* feat: continuous workspace done

* fix remove commented code

* fix: some linting errors

* fix: replace multiple if's by a for

* fix: observations bug, chart titles

* feat: added extra logger graph

* fix: environment imports

* feat: goal in state, logger used

* fix: add actions back, change workspace

* fix: change dqn parameters

* fix: saving dqn model + eps graph

* fix: negative reward for very small movement, add observations to state

* some dqn's

* fix: update robot.urdf to have rotating anchor

* feat: new robot config is used

* fix: remove penalty for not moving

* chore: merge new morphology code

* fix: list index out of range error resolved

* feat: Integrate morphevo with env so modules can rotate and tilt

Co-authored-by: smessie <smessie@smessie.com>

* feat: 2d working dqn

* fix: reorder imports

* fix: pylint errors

* fix: rl now uses run.py

* fix: remove wrong comments

Co-authored-by: Iwijn <iwijn.voeten@ugent.be>
Co-authored-by: Iwijn <iwijn.voeten@gmail.com>
Co-authored-by: smessie <smessie@smessie.com>

File: src/environment/robot.urdf (robot description, URDF)
Before this commit: robot robot, 4 links, 3 joints
Links:
- link MODULE_1: geometry visual tilting_module length=1.5

Commit message: feat: set new workspace and robot arm config

File: src/environment/robot.urdf (robot description, URDF)
Before this commit: robot robot, 4 links, 3 joints
Links:
- added link MODULE_0; visual tilting_module length=1.5
- link MODULE_1: geometry visual tilting_module length=2.5
- link MODULE_2: geometry visual tilting_module length=2.5
- link MODULE_3: geometry visual complex_module length=2.5
- link anchor: geometry visual anchor_module length=1
Joints:
- added joint MODULE_0_JOINT: type revolute, parent MODULE_3, child MODULE_0

Commit message: Change robot colors, add more walls, URDFs and screenshots

File: src/environment/robot.urdf (robot description, URDF)
Before this commit: robot robot, 4 links, 3 joints
Links:
- link MODULE_1: geometry visual complex_module length=1.5
