Commit message: feat: robot urdfs, more fixes

File: src/configs/robots/final_coevolution_robot.urdf (robot description, URDF)
Before this commit: robot robot_-3424064500001286933, 4 links, 3 joints
Links:
- link module_0: geometry visual tilting_module length=0.8549456538724792
- link module_1: geometry visual tilting_module length=2.271242800502206
- link module_2: geometry visual tilting_module length=1.2742207202266767

File: src/configs/robots/halfway_coevolution_robot.urdf (robot description, URDF)
Before this commit: robot robot_6885413710201939357, 4 links, 3 joints
Links:
- link anchor: geometry visual anchor_module length=1.0
- link module_0: geometry visual tilting_module length=0.9889023604622627
- link module_1: geometry visual tilting_module length=0.7621771844608689
- link module_2: geometry visual rotating_module length=2.1204497304575574

File: src/configs/robots/long_robot.urdf (robot description, URDF)
Before this commit: robot robot, 5 links, 4 joints
Links:
- removed link MODULE_4
- link MODULE_1: geometry visual tilting_module length=2.7
- link MODULE_2: geometry visual tilting_module length=2.7
- link MODULE_3: geometry visual tilting_module length=2.7
Joints:
- removed joint MODULE_4_JOINT

File: src/configs/robots/manual_robot.urdf (robot description, URDF)
Before this commit: robot robot, 5 links, 3 joints
Links:
- removed link MODULE_0
- link MODULE_1: geometry visual tilting_module length=1.5
- link MODULE_2: geometry visual tilting_module length=1.5
- link MODULE_3: geometry visual tilting_module length=1.5
- link anchor: geometry visual anchor_module length=0.5
